Commit message: [feat] add gripper for rm75

File: public/urdf/rm75-urdf/urdf/rm_dual.urdf (robot description, URDF)
Before this commit: robot rm_75_dual_description, 25 links, 24 joints
Links:
- removed link left_f_sensor
- removed link left_left_robotiq
- removed link left_right_robotiq
- removed link left_tool_hand
- removed link right_f_sensor
- removed link right_left_robotiq
- removed link right_right_robotiq
- removed link right_tool_hand
- added link left_inner_finger; collision mesh filename=../meshes/robotiq_arg2f_85_inner_finger.dae scale=0.001 0.001 0.001; visual mesh filename=../meshes/robotiq_arg2f_85_inner_finger.dae scale=0.001 0.001 0.001
- added link left_inner_finger_pad; collision box size=0.022 0.00635 0.0375; visual box size=0.022 0.00635 0.0375
- added link left_inner_knuckle; collision mesh filename=../meshes/robotiq_arg2f_85_inner_knuckle.dae scale=0.001 0.001 0.001; visual mesh filename=../meshes/robotiq_arg2f_85_inner_knuckle.dae scale=0.001 0.001 0.001
- added link left_outer_finger; collision mesh filename=../meshes/robotiq_arg2f_85_outer_finger.dae scale=0.001 0.001 0.001; visual mesh filename=../meshes/robotiq_arg2f_85_outer_finger.dae scale=0.001 0.001 0.001
- added link left_outer_knuckle; collision mesh filename=../meshes/robotiq_arg2f_85_outer_knuckle.dae scale=0.001 0.001 0.001; visual mesh filename=../meshes/robotiq_arg2f_85_outer_knuckle.dae scale=0.001 0.001 0.001
- added link left_right_inner_finger; collision mesh filename=../meshes/robotiq_arg2f_85_inner_finger.dae scale=0.001 0.001 0.001; visual mesh filename=../meshes/robotiq_arg2f_85_inner_finger.dae scale=0.001 0.001 0.001
- added link left_right_inner_finger_pad; collision box size=0.022 0.00635 0.0375; visual box size=0.022 0.00635 0.0375
- added link left_right_inner_knuckle; collision mesh filename=../meshes/robotiq_arg2f_85_inner_knuckle.dae scale=0.001 0.001 0.001; visual mesh filename=../meshes/robotiq_arg2f_85_inner_knuckle.dae scale=0.001 0.001 0.001
- added link left_right_outer_finger; collision mesh filename=../meshes/robotiq_arg2f_85_outer_finger.dae scale=0.001 0.001 0.001; visual mesh filename=../meshes/robotiq_arg2f_85_outer_finger.dae scale=0.001 0.001 0.001
- added link left_right_outer_knuckle; collision mesh filename=../meshes/robotiq_arg2f_85_outer_knuckle.dae scale=0.001 0.001 0.001; visual mesh filename=../meshes/robotiq_arg2f_85_outer_knuckle.dae scale=0.001 0.001 0.001
- added link left_robotiq_arg2f_base_link, mass 0.22652; collision mesh filename=../meshes/robotiq_arg2f_base_link.stl; visual mesh filename=../meshes/robotiq_arg2f_base_link.stl
- added link right_inner_finger; collision mesh filename=../meshes/robotiq_arg2f_85_inner_finger.dae scale=0.001 0.001 0.001; visual mesh filename=../meshes/robotiq_arg2f_85_inner_finger.dae scale=0.001 0.001 0.001
- added link right_inner_finger_pad; collision box size=0.022 0.00635 0.0375; visual box size=0.022 0.00635 0.0375
- added link right_inner_knuckle; collision mesh filename=../meshes/robotiq_arg2f_85_inner_knuckle.dae scale=0.001 0.001 0.001; visual mesh filename=../meshes/robotiq_arg2f_85_inner_knuckle.dae scale=0.001 0.001 0.001
- added link right_outer_finger; collision mesh filename=../meshes/robotiq_arg2f_85_outer_finger.dae scale=0.001 0.001 0.001; visual mesh filename=../meshes/robotiq_arg2f_85_outer_finger.dae scale=0.001 0.001 0.001
- added link right_outer_knuckle; collision mesh filename=../meshes/robotiq_arg2f_85_outer_knuckle.dae scale=0.001 0.001 0.001; visual mesh filename=../meshes/robotiq_arg2f_85_outer_knuckle.dae scale=0.001 0.001 0.001
- added link right_right_inner_finger; collision mesh filename=../meshes/robotiq_arg2f_85_inner_finger.dae scale=0.001 0.001 0.001; visual mesh filename=../meshes/robotiq_arg2f_85_inner_finger.dae scale=0.001 0.001 0.001
- added link right_right_inner_finger_pad; collision box size=0.022 0.00635 0.0375; visual box size=0.022 0.00635 0.0375
- added link right_right_inner_knuckle; collision mesh filename=../meshes/robotiq_arg2f_85_inner_knuckle.dae scale=0.001 0.001 0.001; visual mesh filename=../meshes/robotiq_arg2f_85_inner_knuckle.dae scale=0.001 0.001 0.001
- added link right_right_outer_finger; collision mesh filename=../meshes/robotiq_arg2f_85_outer_finger.dae scale=0.001 0.001 0.001; visual mesh filename=../meshes/robotiq_arg2f_85_outer_finger.dae scale=0.001 0.001 0.001
- added link right_right_outer_knuckle; collision mesh filename=../meshes/robotiq_arg2f_85_outer_knuckle.dae scale=0.001 0.001 0.001; visual mesh filename=../meshes/robotiq_arg2f_85_outer_knuckle.dae scale=0.001 0.001 0.001
- added link right_robotiq_arg2f_base_link, mass 0.22652; collision mesh filename=../meshes/robotiq_arg2f_base_link.stl; visual mesh filename=../meshes/robotiq_arg2f_base_link.stl
Joints:
- removed joint left_joint_f_sensor
- removed joint left_joint_hand
- removed joint left_left_joint_robotiq
- removed joint left_right_joint_robotiq
- removed joint right_joint_f_sensor
- removed joint right_joint_hand
- removed joint right_left_joint_robotiq
- removed joint right_right_joint_robotiq
- added joint left_finger_joint: type revolute, parent left_robotiq_arg2f_base_link, child left_outer_knuckle, origin xyz=0 -0.0306011 0.054904 rpy=0 0 3.141592653589793, axis 1 0 0, limit lower=0 upper=0.8 effort=1000 velocity=2.0
- added joint left_gripper_base_joint: type fixed, parent left_Link7, child left_robotiq_arg2f_base_link, origin xyz=0 0 0 rpy=0 0 1.57
- added joint left_inner_finger_joint: type revolute, parent left_outer_finger, child left_inner_finger, origin xyz=0 0.0061 0.0471 rpy=0 0 0, axis 1 0 0, limit lower=0 upper=0.8757 effort=1000 velocity=2.0, mimic joint=left_finger_joint multiplier=-1 offset=0
- added joint left_inner_finger_pad_joint: type fixed, parent left_inner_finger, child left_inner_finger_pad, origin xyz=0 -0.0220203446692936 0.03242 rpy=0 0 0, axis 0 0 1
- added joint left_inner_knuckle_joint: type revolute, parent left_robotiq_arg2f_base_link, child left_inner_knuckle, origin xyz=0 -0.0127 0.06142 rpy=0 0 3.141592653589793, axis 1 0 0, limit lower=0 upper=0.8757 effort=1000 velocity=2.0, mimic joint=left_finger_joint multiplier=1 offset=0
- added joint left_outer_finger_joint: type fixed, parent left_outer_knuckle, child left_outer_finger, origin xyz=0 0.0315 -0.0041 rpy=0 0 0, axis 1 0 0
- added joint left_right_inner_finger_joint: type revolute, parent left_right_outer_finger, child left_right_inner_finger, origin xyz=0 0.0061 0.0471 rpy=0 0 0, axis 1 0 0, limit lower=0 upper=0.8757 effort=1000 velocity=2.0, mimic joint=left_finger_joint multiplier=-1 offset=0
- added joint left_right_inner_finger_pad_joint: type fixed, parent left_right_inner_finger, child left_right_inner_finger_pad, origin xyz=0 -0.0220203446692936 0.03242 rpy=0 0 0, axis 0 0 1
- added joint left_right_inner_knuckle_joint: type revolute, parent left_robotiq_arg2f_base_link, child left_right_inner_knuckle, origin xyz=0 0.0127 0.06142 rpy=0 0 0.0, axis 1 0 0, limit lower=0 upper=0.8757 effort=1000 velocity=2.0, mimic joint=left_finger_joint multiplier=1 offset=0
- added joint left_right_outer_finger_joint: type fixed, parent left_right_outer_knuckle, child left_right_outer_finger, origin xyz=0 0.0315 -0.0041 rpy=0 0 0, axis 1 0 0
- added joint left_right_outer_knuckle_joint: type revolute, parent left_robotiq_arg2f_base_link, child left_right_outer_knuckle, origin xyz=0 0.0306011 0.054904 rpy=0 0 0, axis 1 0 0, limit lower=0 upper=0.81 effort=1000 velocity=2.0, mimic joint=left_finger_joint multiplier=1 offset=0
- added joint right_finger_joint: type revolute, parent right_robotiq_arg2f_base_link, child right_outer_knuckle, origin xyz=0 -0.0306011 0.054904 rpy=0 0 3.141592653589793, axis 1 0 0, limit lower=0 upper=0.8 effort=1000 velocity=2.0
- added joint right_gripper_base_joint: type fixed, parent right_Link7, child right_robotiq_arg2f_base_link, origin xyz=0 0 0 rpy=0 0 1.57
- added joint right_inner_finger_joint: type revolute, parent right_outer_finger, child right_inner_finger, origin xyz=0 0.0061 0.0471 rpy=0 0 0, axis 1 0 0, limit lower=0 upper=0.8757 effort=1000 velocity=2.0, mimic joint=right_finger_joint multiplier=-1 offset=0
- added joint right_inner_finger_pad_joint: type fixed, parent right_inner_finger, child right_inner_finger_pad, origin xyz=0 -0.0220203446692936 0.03242 rpy=0 0 0, axis 0 0 1
- added joint right_inner_knuckle_joint: type revolute, parent right_robotiq_arg2f_base_link, child right_inner_knuckle, origin xyz=0 -0.0127 0.06142 rpy=0 0 3.141592653589793, axis 1 0 0, limit lower=0 upper=0.8757 effort=1000 velocity=2.0, mimic joint=right_finger_joint multiplier=1 offset=0
- added joint right_outer_finger_joint: type fixed, parent right_outer_knuckle, child right_outer_finger, origin xyz=0 0.0315 -0.0041 rpy=0 0 0, axis 1 0 0
- added joint right_right_inner_finger_joint: type revolute, parent right_right_outer_finger, child right_right_inner_finger, origin xyz=0 0.0061 0.0471 rpy=0 0 0, axis 1 0 0, limit lower=0 upper=0.8757 effort=1000 velocity=2.0, mimic joint=right_finger_joint multiplier=-1 offset=0
- added joint right_right_inner_finger_pad_joint: type fixed, parent right_right_inner_finger, child right_right_inner_finger_pad, origin xyz=0 -0.0220203446692936 0.03242 rpy=0 0 0, axis 0 0 1
- added joint right_right_inner_knuckle_joint: type revolute, parent right_robotiq_arg2f_base_link, child right_right_inner_knuckle, origin xyz=0 0.0127 0.06142 rpy=0 0 0.0, axis 1 0 0, limit lower=0 upper=0.8757 effort=1000 velocity=2.0, mimic joint=right_finger_joint multiplier=1 offset=0
- added joint right_right_outer_finger_joint: type fixed, parent right_right_outer_knuckle, child right_right_outer_finger, origin xyz=0 0.0315 -0.0041 rpy=0 0 0, axis 1 0 0
- added joint right_right_outer_knuckle_joint: type revolute, parent right_robotiq_arg2f_base_link, child right_right_outer_knuckle, origin xyz=0 0.0306011 0.054904 rpy=0 0 0, axis 1 0 0, limit lower=0 upper=0.81 effort=1000 velocity=2.0, mimic joint=right_finger_joint multiplier=1 offset=0
- joint left_base_mounting_joint: origin xyz=0 0.1 0 rpy=-1.5708 -1.5708 -0.4363 -> xyz=0 0.025 0 rpy=-1.5708 -1.5708 -0.4363
- joint right_base_mounting_joint: origin xyz=0 -0.1 0 rpy=1.5708 -1.5708 0.4363 -> xyz=0 -0.025 0 rpy=1.5708 -1.5708 0.4363
